File: RotaryEncoder/RotaryEncoder.sch (EAGLE design)
At the start: 21 parts, among them Q1 MOSFET-NCHANNELBSS138, Q2 MOSFET-NCHANNELBSS138

Commit message: Latest version of schematics and boards
Parts:
- removed C2: .47uF, SparkFun-Capacitors:CAP0805
- removed C3, C4: 2.2uF, SparkFun-Capacitors:CAP0805
- removed C5, C6: 1uF, SparkFun-Capacitors:CAP0805
- removed Q1, Q2: MOSFET-NCHANNELBSS138, SparkFun-DiscreteSemi:MOSFET-NCHANNELBSS138
- removed U$2: 3.3V/150mA, SparkFun-PowerIC:V_REG_MIC52053.3V
- removed U$3, U$4, U$6: KMR441G, IntegerLabs:TACT-SWITCHKMR2
- removed U$8: ATTINY48/88-TQFP, IntegerLabs:ATTINY48/88-TQFP
- added R6: 2k, SparkFun-Passives:RESISTOR0805-RES
- added SW1: (no value), SparkFun-Electromechanical:ENCODER_RGB_CA
- R1: value 390k -> 120
- R3, R4: value 2k -> 68
- U$1: value OLEDREVERSE -> TINY841; device IntegerLabs:OLEDREVERSE -> IntegerLabs:TINY841
Connections:
- removed net +3.3V: C2.1, Q1.G, Q2.G, R3.2, R4.2, U$1.BS2, U$1.VBAT, U$1.VDD, U$2.OUT, U$7.VPROG, U$8.AVCC, U$8.VCC
- removed net +5V: C1.2, R5.1, U$2.EN, U$2.IN
- removed net BS1: U$1.BS1, U$8.PC1
- removed net BUTTON0: U$3.POS1, U$8.PA0
- removed net BUTTON1: U$6.POS1, U$8.PA1
- removed net BUTTON2: U$4.POS1, U$8.PA2
- removed net CS: U$1.CS, U$8.PB6
- removed net D/C: U$1.D/C, U$8.PB7
- removed net D0: U$1.D0, U$8.PD0
- removed net D1: U$1.D1, U$8.PD1
- removed net D2: U$1.D2, U$8.PD2
- removed net D3: U$1.D3, U$8.PD3
- removed net D4: U$1.D4, U$8.PD4
- removed net D5: U$1.D5, U$8.PD5
- removed net D6: U$1.D6, U$8.PD6
- removed net D7: U$1.D7, U$8.PD7
- removed net DISPLAY_RESET: U$1.RESET, U$8.PA3
- removed net E/RD: U$1.E/RD, U$8.PB0
- removed net MOSI: U$7.MOSI, U$8.PB3
- removed net N$10: C6.2, U$1.C2P
- removed net N$11: C5.1, U$1.C1N
- removed net N$12: C6.1, U$1.C2N
- removed net N$2: R1.2, U$1.IREF
- removed net N$9: C5.2, U$1.C1P
- removed net R/W: U$1.R/W, U$8.PC3
- removed net SCK: U$7.SCK, U$8.PB5
- removed net SCL: Q1.D, U$7.SCL
- removed net SCL3.3: Q1.S, R3.1, U$8.PC5
- removed net SDA3.3: Q2.S, R4.1, U$8.PC4
- new net A: SW1.A, U$1.PB0
- new net B: SW1.B, U$1.PB1
- new net BLUE: R4.2, U$1.PA3
- new net GREEN: R3.2, U$1.PA2
- new net N$5: R3.1, SW1.-G
- new net RED: R1.2, U$1.PA1
- new net SCL/SCK: U$1.PA4, U$7.SCK, U$7.SCL
- new net SDA/MOSI: U$1.PA6, U$7.MOSI
- new net SW: R6.1, SW1.SW, U$1.PB2
- new net VCC: C1.2, R5.1, SW1.+, U$1.VCC, U$7.VPROG
- net GND: now also R6.2, SW1.C, U$1.GND; no longer C2.2, C3.2, C4.2, R1.1, U$1.BS0, U$1.VLSS, U$1.VSS, U$2.GND, U$3.NEG1, U$3.NEG2, U$4.NEG1, U$4.NEG2, U$6.NEG1, U$6.NEG2, U$8.GND, U$8.GND@1
- net LED: now also U$1.PA7; no longer U$8.PB1
- net MISO: now also U$1.PA5; no longer U$8.PB4
- net N$4: now also R1.1, SW1.-R; no longer C3.1, U$1.VCC
- net N$6: now also R4.1, SW1.-B; no longer C4.1, U$1.VCOMH
- net RESET: now also U$1.PB3; no longer U$8.PC6
- net SDA: no longer Q2.D
Other:
- moved on the sheet: C1, LED1, R1, R2, R3, R4, R5

Commit message: New versions of IntegerLabs library, RotaryEncoder, and Thermocouple
Connections:
- removed net SDA: U$7.SDA
- net SDA/MOSI: now also U$7.SDA
Changed lines of the file:
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@@
 <label x="73.66" y="10.16" size="1.778" layer="95"/>
+</segment>
+<segment>
+<pinref part="U$7" gate="G$1" pin="SDA"/>
+<wire x1="43.18" y1="33.02" x2="30.48" y2="33.02" width="0.1524" layer="91"/>
+<label x="30.48" y="33.02" size="1.778" layer="95"/>
 </segment>
 </net>
@@
 </segment>
 </net>
-<net name="SDA" class="0">
-<segment>
-<pinref part="U$7" gate="G$1" pin="SDA"/>
-<wire x1="43.18" y1="33.02" x2="35.56" y2="33.02" width="0.1524" layer="91"/>
-<label x="35.56" y="33.02" size="1.778" layer="95"/>
-</segment>
-</net>
