File: GPIO/GPIO.sch (EAGLE design)
At the start: 29 parts

Commit message: Checkpointing PCB designs
Parts:
- added C1, C3: (no value), SparkFun-Capacitors:CAP1206
- JP2: device SparkFun-Connectors:M10NO_SILK -> SparkFun-Connectors:M08NO_SILK
- LED: device led:LEDCHIPLED_1206 -> adafruit:LEDCHIPLED_0805
- R10, R11, R12, R13, R14, R15, R8, R9: value 200 -> 130
- U$4: BOARD (none) -> I/O; VERSION (none) -> v6
Connections:
- net GND: now also C1.1, C3.1; no longer JP2.10
- net VOUT: now also C1.2, C3.2; no longer JP2.9
Changed lines of the file:
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@@
 <layers>
 <layer number="1" name="Top" color="4" fill="1" visible="no" active="no"/>
+<layer number="2" name="Route2" color="1" fill="3" visible="no" active="no"/>
+<layer number="3" name="Route3" color="4" fill="3" visible="no" active="no"/>
+<layer number="14" name="Route14" color="1" fill="6" visible="no" active="no"/>
+<layer number="15" name="Route15" color="4" fill="6" visible="no" active="no"/>
 <layer number="16" name="Bottom" color="1" fill="1" visible="no" active="no"/>
 <layer number="17" name="Pads" color="2" fill="1" visible="no" active="no"/>
@@
 <part name="C2" library="SparkFun-Capacitors" deviceset="CAP" device="0805" value=".47uF"/>
 <part name="RLED" library="SparkFun-Passives" deviceset="RESISTOR" device="0805-RES" value="680"/>
-<part name="LED" library="led" deviceset="LED" device="CHIPLED_1206" value="blue"/>
+<part name="LED" library="adafruit" deviceset="LED" device="CHIPLED_0805" value="blue"/>
 <part name="U$3" library="IntegerLabs" deviceset="TINY841" device=""/>
-<part name="U$4" library="IntegerLabs" deviceset="FOOTPRINT" device="FOOTPRINT-2" value="FOOTPRINTFOOTPRINT-2"/>
-<part name="JP2" library="SparkFun-Connectors" deviceset="M10" device="NO_SILK" value="M10NO_SILK"/>
+<part name="U$4" library="IntegerLabs" deviceset="FOOTPRINT" device="FOOTPRINT-2" value="FOOTPRINTFOOTPRINT-2">
+<attribute name="BOARD" value="I/O"/>
+<attribute name="VERSION" value="v6"/>
+</part>
+<part name="JP2" library="SparkFun-Connectors" deviceset="M08" device="NO_SILK" value="M10NO_SILK"/>
 <part name="JP1" library="SparkFun-Connectors" deviceset="M08" device="NO_SILK"/>
 <part name="JP3" library="SparkFun-Connectors" deviceset="M08" device="NO_SILK"/>
@@
 <part name="R6" library="SparkFun-Passives" deviceset="SOLDERJUMPER" device="NO"/>
 <part name="R7" library="SparkFun-Passives" deviceset="SOLDERJUMPER" device="NO"/>
-<part name="R8" library="SparkFun-Resistors" deviceset="RESISTOR" device="0805-RES" value="200"/>
-<part name="R9" library="SparkFun-Resistors" deviceset="RESISTOR" device="0805-RES" value="200"/>
-<part name="R10" library="SparkFun-Resistors" deviceset="RESISTOR" device="0805-RES" value="200"/>
-<part name="R11" library="SparkFun-Resistors" deviceset="RESISTOR" device="0805-RES" value="200"/>
-<part name="R12" library="SparkFun-Resistors" deviceset="RESISTOR" device="0805-RES" value="200"/>
-<part name="R13" library="SparkFun-Resistors" deviceset="RESISTOR" device="0805-RES" value="200"/>
-<part name="R14" library="SparkFun-Resistors" deviceset="RESISTOR" device="0805-RES" value="200"/>
-<part name="R15" library="SparkFun-Resistors" deviceset="RESISTOR" device="0805-RES" value="200"/>
+<part name="R8" library="SparkFun-Resistors" deviceset="RESISTOR" device="0805-RES" value="130"/>
+<part name="R9" library="SparkFun-Resistors" deviceset="RESISTOR" device="0805-RES" value="130"/>
+<part name="R10" library="SparkFun-Resistors" deviceset="RESISTOR" device="0805-RES" value="130"/>
+<part name="R11" library="SparkFun-Resistors" deviceset="RESISTOR" device="0805-RES" value="130"/>
+<part name="R12" library="SparkFun-Resistors" deviceset="RESISTOR" device="0805-RES" value="130"/>
+<part name="R13" library="SparkFun-Resistors" deviceset="RESISTOR" device="0805-RES" value="130"/>
+<part name="R14" library="SparkFun-Resistors" deviceset="RESISTOR" device="0805-RES" value="130"/>
+<part name="R15" library="SparkFun-Resistors" deviceset="RESISTOR" device="0805-RES" value="130"/>
 <part name="D26" library="diode" deviceset="BAS70XY" device=""/>
 <part name="D27" library="diode" deviceset="BAS70XY" device=""/>
 <part name="D28" library="diode" deviceset="BAS70XY" device=""/>
 <part name="D29" library="diode" deviceset="BAS70XY" device=""/>
+<part name="C1" library="SparkFun-Capacitors" deviceset="CAP" device="1206"/>
+<part name="C3" library="SparkFun-Capacitors" deviceset="CAP" device="1206"/>
 </parts>
 <sheets>
@@
 <instance part="U$3" gate="G$1" x="33.02" y="12.7"/>
 <instance part="U$4" gate="G$1" x="162.56" y="7.62"/>
-<instance part="JP2" gate="G$1" x="50.8" y="68.58"/>
+<instance part="JP2" gate="G$1" x="53.34" y="58.42"/>
 <instance part="JP1" gate="G$1" x="15.24" y="68.58"/>
 <instance part="JP3" gate="G$1" x="38.1" y="68.58"/>
@@
 <instance part="D29" gate="A" x="236.22" y="17.78"/>
 <instance part="D29" gate="B" x="274.32" y="17.78"/>
+<instance part="C1" gate="G$1" x="43.18" y="101.6"/>
+<instance part="C3" gate="G$1" x="48.26" y="101.6"/>
 </instances>
 <busses>
@@
 <wire x1="152.4" y1="22.86" x2="134.62" y2="22.86" width="0.1524" layer="91"/>
 <label x="134.62" y="22.86" size="1.778" layer="95"/>
-</segment>
-<segment>
-<pinref part="JP2" gate="G$1" pin="10"/>
-<wire x1="60.96" y1="73.66" x2="66.04" y2="73.66" width="0.1524" layer="91"/>
-<label x="60.96" y="73.66" size="1.778" layer="95"/>
 </segment>
 <segment>
@@
 <label x="259.08" y="17.78" size="1.778" layer="95"/>
 </segment>
+<segment>
+<pinref part="C3" gate="G$1" pin="1"/>
+<pinref part="C1" gate="G$1" pin="1"/>
+<wire x1="48.26" y1="106.68" x2="43.18" y2="106.68" width="0.1524" layer="91"/>
+<wire x1="43.18" y1="106.68" x2="35.56" y2="106.68" width="0.1524" layer="91"/>
+<label x="35.56" y="106.68" size="1.778" layer="95"/>
+</segment>
 </net>
 <net name="RESET" class="0">
@@
 <segment>
 <pinref part="JP2" gate="G$1" pin="1"/>
-<wire x1="60.96" y1="50.8" x2="66.04" y2="50.8" width="0.1524" layer="91"/>
+<wire x1="58.42" y1="50.8" x2="66.04" y2="50.8" width="0.1524" layer="91"/>
 <label x="60.96" y="50.8" size="1.778" layer="95"/>
 </segment>
@@
 <segment>
 <pinref part="JP2" gate="G$1" pin="2"/>
-<wire x1="60.96" y1="53.34" x2="66.04" y2="53.34" width="0.1524" layer="91"/>
+<wire x1="58.42" y1="53.34" x2="66.04" y2="53.34" width="0.1524" layer="91"/>
 <label x="60.96" y="53.34" size="1.778" layer="95"/>
 </segment>
@@
 <segment>
 <pinref part="JP2" gate="G$1" pin="3"/>
-<wire x1="60.96" y1="55.88" x2="66.04" y2="55.88" width="0.1524" layer="91"/>
+<wire x1="58.42" y1="55.88" x2="66.04" y2="55.88" width="0.1524" layer="91"/>
 <label x="60.96" y="55.88" size="1.778" layer="95"/>
 </segment>
@@
 <segment>
 <pinref part="JP2" gate="G$1" pin="4"/>
-<wire x1="60.96" y1="58.42" x2="66.04" y2="58.42" width="0.1524" layer="91"/>
+<wire x1="58.42" y1="58.42" x2="66.04" y2="58.42" width="0.1524" layer="91"/>
 <label x="60.96" y="58.42" size="1.778" layer="95"/>
 </segment>
@@
 <segment>
 <pinref part="JP2" gate="G$1" pin="5"/>
-<wire x1="60.96" y1="60.96" x2="66.04" y2="60.96" width="0.1524" layer="91"/>
+<wire x1="58.42" y1="60.96" x2="66.04" y2="60.96" width="0.1524" layer="91"/>
 <label x="60.96" y="60.96" size="1.778" layer="95"/>
 </segment>
@@
 <segment>
 <pinref part="JP2" gate="G$1" pin="6"/>
-<wire x1="60.96" y1="63.5" x2="66.04" y2="63.5" width="0.1524" layer="91"/>
+<wire x1="58.42" y1="63.5" x2="66.04" y2="63.5" width="0.1524" layer="91"/>
 <label x="60.96" y="63.5" size="1.778" layer="95"/>
 </segment>
@@
 <segment>
 <pinref part="JP2" gate="G$1" pin="7"/>
-<wire x1="60.96" y1="66.04" x2="66.04" y2="66.04" width="0.1524" layer="91"/>
+<wire x1="58.42" y1="66.04" x2="66.04" y2="66.04" width="0.1524" layer="91"/>
 <label x="60.96" y="66.04" size="1.778" layer="95"/>
 </segment>
@@
 <segment>
 <pinref part="JP2" gate="G$1" pin="8"/>
-<wire x1="60.96" y1="68.58" x2="66.04" y2="68.58" width="0.1524" layer="91"/>
+<wire x1="58.42" y1="68.58" x2="66.04" y2="68.58" width="0.1524" layer="91"/>
 <label x="60.96" y="68.58" size="1.778" layer="95"/>
 </segment>
@@
 <pinref part="JP3" gate="G$1" pin="1"/>
 <wire x1="43.18" y1="63.5" x2="43.18" y2="60.96" width="0.1524" layer="91"/>
-<pinref part="JP2" gate="G$1" pin="9"/>
-<wire x1="60.96" y1="71.12" x2="68.58" y2="71.12" width="0.1524" layer="91"/>
-<wire x1="68.58" y1="71.12" x2="68.58" y2="81.28" width="0.1524" layer="91"/>
-<wire x1="68.58" y1="81.28" x2="43.18" y2="81.28" width="0.1524" layer="91"/>
-<wire x1="43.18" y1="81.28" x2="43.18" y2="78.74" width="0.1524" layer="91"/>
-<wire x1="43.18" y1="81.28" x2="43.18" y2="91.44" width="0.1524" layer="91"/>
+<wire x1="43.18" y1="78.74" x2="43.18" y2="91.44" width="0.1524" layer="91"/>
 <pinref part="D1" gate="G$1" pin="C"/>
-<wire x1="43.18" y1="91.44" x2="50.8" y2="91.44" width="0.1524" layer="91"/>
-</segment>
-</net>
+<wire x1="43.18" y1="91.44" x2="48.26" y2="91.44" width="0.1524" layer="91"/>
+<pinref part="C1" gate="G$1" pin="2"/>
+<wire x1="48.26" y1="91.44" x2="50.8" y2="91.44" width="0.1524" layer="91"/>
+<wire x1="43.18" y1="99.06" x2="43.18" y2="91.44" width="0.1524" layer="91"/>
+<pinref part="C3" gate="G$1" pin="2"/>
+<wire x1="48.26" y1="99.06" x2="48.26" y2="91.44" width="0.1524" layer="91"/>
+</segment>
+</net>
