File: MagController/MagController.sch (EAGLE design)
At the start: 40 parts, among them Q1 16Mhz, Q2 DMMT5401, Q3 DMG2305UX

Commit message: Checkpointing PCB designs
Parts:
- removed C6: 10uF, SparkFun-Capacitors:CAP0805
- removed FOOTPRINT: Controller, IntegerLabs:FOOTPRINTFOOTPRINT-2
- removed JP1, JP2, JP3: (no value), adafruit:PINHD-1X6LOCK
- removed Q2: DMMT5401, IntegerLabs:TRANSISTOR-DUAL-PNP
- removed Q3: DMG2305UX, transistor-power:IRLML5203
- removed R17, R18: 130, SparkFun-Resistors:RESISTOR0805-RES
- removed R8: 2k, SparkFun-Resistors:RESISTOR0805-RES
- removed R9: 47k 1%, SparkFun-Passives:RESISTOR0805-RES
- removed SJ1: SOLDERJUMPERNO, SparkFun-Passives:SOLDERJUMPERNO
- removed U$4: USBFCI-MICROB, IntegerLabs:USBFCI-MICROB
- removed U$6: TACT-SWITCHBOURNS-7914J, IntegerLabs:TACT-SWITCHBOURNS-7914J
- added C8: 100nF, Modulo:CAPACITOR-100NF
- added D1: (no value), SparkFun-DiscreteSemi:DIODESMA
- added JP4, JP5, JP6: (no value), SparkFun-Connectors:M05NO_SILK
- added L1: 10uH, Modulo:INDUCTOR-10UH
- added PCB1: MAGDEVICE, Modulo:MAGDEVICE
- added SW1: blue, Modulo:SWITCHBOURNS-7914J
- added U3: USBFCI-MICROB, IntegerLabs:USBFCI-MICROB
- C1: device SparkFun-Capacitors:CAP0805 -> Modulo:CAPACITOR-1UF
- C2, C3: device SparkFun-Capacitors:CAP0805 -> Modulo:CAPACITOR-18PF
- C4, C7: value .47uF -> 100nF; device SparkFun-Capacitors:CAP0805 -> Modulo:CAPACITOR-100NF
- C5: value 47uF -> 10uF; device SparkFun-Capacitors:CAP1206 -> Modulo:CAPACITOR-10UF
- F1: value MF-PSMF110X-2 -> 2A; device SparkFun-Resistors:RESISTOR0805-RES -> Modulo:RESISTOR-0603; PARTNUM (none) -> MF-PSMF110X-2
- LED1: value (none) -> blue; device adafruit:LEDCHIP-LED0805 -> Modulo:LED-0805-BLUE
- LED2: value (none) -> green; device led:LEDCHIPLED_0805 -> Modulo:LED-0805-GREEN
- Q1: device adafruit:XTAL-4-3225 -> Modulo:CRYSTAL-NX3225; PARTNUM (none) -> CX3225GB16000P0HPQCC
- R1, R10, R11, R12, R2: value 2k -> 1.5KΩ; device SparkFun-Resistors:RESISTOR0805-RES -> Modulo:RESISTOR-1.5KΩ
- R13, R14, R15, R16: value 130 -> 150Ω; device SparkFun-Resistors:RESISTOR0805-RES -> Modulo:RESISTOR-150Ω
- R3, R4: value 22 -> 22Ω; device SparkFun-Resistors:RESISTOR0805-RES -> Modulo:RESISTOR-22Ω
- R5: value 10k 1% -> 150Ω; device SparkFun-Passives:RESISTOR0805-RES -> Modulo:RESISTOR-150Ω
- R6, R7: value 680 -> 681Ω; device SparkFun-Resistors:RESISTOR0805-RES -> Modulo:RESISTOR-681Ω
- U1: PARTNUM (none) -> ATMEGA32U4-AU
- U2: PARTNUM (none) -> MIC5205-3.3YM5 TR
- renumbered U$1 to U2, U$2 to U1
Connections:
- removed net D1: R17.1, R8.2, U1.PC6
- removed net MOSI: FOOTPRINT.MOSI, U1.PB2(MOSI)
- removed net N$14: Q2A.B, Q2A.C, Q2B.B, R5.2
- removed net N$16: Q2B.C, Q3.G, R9.2
- removed net N$19: JP1.5, R17.2
- removed net N$20: JP1.6, R18.2
- removed net SCK: FOOTPRINT.SCK, U1.PB1(SCK)
- new net AVCC: C8.1, L1.2, U1.AVCC@24, U1.AVCC@44
- net +3.3V: no longer SJ1.2
- net D+: now also U3.D+; no longer U$4.D+
- net D-: now also U3.D-; no longer U$4.D-
- net D0: now also R5.1; no longer R18.1
- net GND: now also C8.2, JP5.1, JP5.2, JP5.3, JP5.4, JP5.5, PCB1.GND, Q1.G1, Q1.G2, SW1.NEG1, U3.GND; no longer C6.2, FOOTPRINT.GND, JP2.1, JP2.2, JP2.3, JP2.4, JP2.5, JP2.6, R5.1, R9.1, U$4.GND, U$6.NEG1
- net MISO: now also PCB1.MISO; no longer FOOTPRINT.MISO
- net N$11: now also JP4.5, R5.2; no longer R8.1, U1.PF7(ADC7)
- net N$13: now also JP4.2; no longer JP1.2
- net N$17: now also JP4.3; no longer JP1.3
- net N$18: now also JP4.4; no longer JP1.4
- net N$2: now also JP4.1; no longer JP1.1
- net N$3: now also U3.VBUS; no longer U$4.VBUS
- net RESET: now also PCB1.RESET, SW1.POS1; no longer FOOTPRINT.RESET, U$6.POS1
- net SCL: now also PCB1.SCL/SCK, U1.PB1(SCK); no longer FOOTPRINT.SCL
- net SDA: now also PCB1.SDA/MOSI, U1.PB2(MOSI); no longer FOOTPRINT.SDA
- net VBUS: now also D1.A; no longer C6.1, Q2A.E, Q3.D, U1.VBUS
- net VCC: now also D1.C, JP6.1, JP6.2, JP6.3, JP6.4, JP6.5, L1.1, PCB1.VCC, PCB1.VPROG, U1.VBUS; no longer FOOTPRINT.VCC, FOOTPRINT.VPROG, JP3.1, JP3.2, JP3.3, JP3.4, JP3.5, JP3.6, Q2B.E, Q3.S, SJ1.1, U1.AVCC@24, U1.AVCC@44
Other:
- moved on the sheet: F1, R1, R2, R5
