File: MagKnob/Knob.sch (EAGLE design)
At the start: 10 parts, among them SW1 TopUp EC12PLRGBSDVBF-D, U1 attiny841-ssur, U2 EXCLUDE

Commit message: Checkpointing PCB designs
Parts:
- removed U2: EXCLUDE, Modulo:DEVICE-PCB
- added PCB1: MAGDEVICE, Modulo:MAGDEVICE
Connections:
- net GND: now also PCB1.GND; no longer U2.GND
- net MISO: now also PCB1.MISO; no longer U2.MISO
- net RESET: now also PCB1.RESET; no longer U2.RESET
- net SCL/SCK: now also PCB1.SCL/SCK; no longer U2.SCK, U2.SCL
- net SDA/MOSI: now also PCB1.SDA/MOSI; no longer U2.MOSI, U2.SDA
- net VCC: now also PCB1.VCC, PCB1.VPROG; no longer U2.VCC, U2.VPROG
Changed lines of the file:
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@@
 <parts>
 <part name="R2" library="Modulo" deviceset="RESISTOR" device="" value="680"/>
-<part name="U2" library="Modulo" deviceset="DEVICE-PCB" device="" value="EXCLUDE">
-<attribute name="NOBOM" value="1"/>
-</part>
 <part name="LED1" library="Modulo" deviceset="LED" device="-0805-BLUE" value="LTST-C171TBKT"/>
 <part name="SW1" library="SparkFun-Electromechanical" deviceset="ENCODER_RGB_CA" device="" value="TopUp EC12PLRGBSDVBF-D"/>
@@
 <part name="P+1" library="supply1" deviceset="VCC" device=""/>
 <part name="C2" library="Modulo" deviceset="CAPACITOR" device="" value=".47uF"/>
+<part name="PCB1" library="Modulo" deviceset="MAGDEVICE" device=""/>
 </parts>
 <sheets>
@@
 <instances>
 <instance part="R2" gate="G$1" x="190.5" y="71.12" rot="R180"/>
-<instance part="U2" gate="G$1" x="71.12" y="83.82">
-<attribute name="NOBOM" x="71.12" y="83.82" size="1.778" layer="96" display="off"/>
-</instance>
 <instance part="LED1" gate="G$1" x="200.66" y="71.12" rot="R90"/>
 <instance part="SW1" gate="G$1" x="193.04" y="99.06"/>
@@
 <attribute name="VALUE" x="72.898" y="109.347" size="1.778" layer="96" rot="R180"/>
 </instance>
+<instance part="PCB1" gate="G$1" x="73.66" y="81.28"/>
 </instances>
 <busses>
@@
 <net name="GND" class="0">
 <segment>
-<pinref part="U2" gate="G$1" pin="GND"/>
-<wire x1="58.42" y1="76.2" x2="55.88" y2="76.2" width="0.1524" layer="91"/>
 <pinref part="GND2" gate="1" pin="GND"/>
 <wire x1="55.88" y1="73.66" x2="55.88" y2="76.2" width="0.1524" layer="91"/>
+<pinref part="PCB1" gate="G$1" pin="GND"/>
+<wire x1="55.88" y1="76.2" x2="58.42" y2="76.2" width="0.1524" layer="91"/>
 </segment>
 <segment>
@@
 <segment>
 <pinref part="U1" gate="G$1" pin="PB3"/>
-<pinref part="U2" gate="G$1" pin="RESET"/>
 <wire x1="99.06" y1="86.36" x2="88.9" y2="86.36" width="0.1524" layer="91"/>
+<pinref part="PCB1" gate="G$1" pin="RESET"/>
 </segment>
 </net>
 <net name="SDA/MOSI" class="0">
 <segment>
-<pinref part="U2" gate="G$1" pin="SDA"/>
 <pinref part="U1" gate="G$1" pin="PA6"/>
-<wire x1="99.06" y1="81.28" x2="96.52" y2="81.28" width="0.1524" layer="91"/>
-<wire x1="96.52" y1="81.28" x2="96.52" y2="78.74" width="0.1524" layer="91"/>
-<pinref part="U2" gate="G$1" pin="MOSI"/>
-<wire x1="96.52" y1="78.74" x2="88.9" y2="78.74" width="0.1524" layer="91"/>
-<wire x1="88.9" y1="76.2" x2="96.52" y2="76.2" width="0.1524" layer="91"/>
-<wire x1="96.52" y1="76.2" x2="96.52" y2="78.74" width="0.1524" layer="91"/>
+<pinref part="PCB1" gate="G$1" pin="SDA/MOSI"/>
+<wire x1="99.06" y1="81.28" x2="88.9" y2="81.28" width="0.1524" layer="91"/>
 </segment>
 </net>
@@
 <segment>
 <pinref part="U1" gate="G$1" pin="PA5"/>
-<pinref part="U2" gate="G$1" pin="MISO"/>
 <wire x1="99.06" y1="88.9" x2="88.9" y2="88.9" width="0.1524" layer="91"/>
+<pinref part="PCB1" gate="G$1" pin="MISO"/>
 </segment>
 </net>
 <net name="SCL/SCK" class="0">
 <segment>
-<pinref part="U2" gate="G$1" pin="SCL"/>
-<wire x1="88.9" y1="81.28" x2="93.98" y2="81.28" width="0.1524" layer="91"/>
 <pinref part="U1" gate="G$1" pin="PA4"/>
-<pinref part="U2" gate="G$1" pin="SCK"/>
-<wire x1="99.06" y1="83.82" x2="93.98" y2="83.82" width="0.1524" layer="91"/>
-<wire x1="93.98" y1="83.82" x2="88.9" y2="83.82" width="0.1524" layer="91"/>
-<wire x1="93.98" y1="81.28" x2="93.98" y2="83.82" width="0.1524" layer="91"/>
+<wire x1="99.06" y1="83.82" x2="88.9" y2="83.82" width="0.1524" layer="91"/>
+<pinref part="PCB1" gate="G$1" pin="SCL/SCK"/>
 </segment>
 </net>
@@
 <net name="VCC" class="0">
 <segment>
-<pinref part="U2" gate="G$1" pin="VPROG"/>
-<pinref part="U2" gate="G$1" pin="VCC"/>
-<wire x1="55.88" y1="88.9" x2="58.42" y2="88.9" width="0.1524" layer="91"/>
+<pinref part="P+1" gate="VCC" pin="VCC"/>
+<wire x1="55.88" y1="86.36" x2="55.88" y2="88.9" width="0.1524" layer="91"/>
+<pinref part="PCB1" gate="G$1" pin="VPROG"/>
+<wire x1="55.88" y1="88.9" x2="55.88" y2="93.98" width="0.1524" layer="91"/>
 <wire x1="58.42" y1="86.36" x2="55.88" y2="86.36" width="0.1524" layer="91"/>
-<wire x1="55.88" y1="86.36" x2="55.88" y2="88.9" width="0.1524" layer="91"/>
-<pinref part="P+1" gate="VCC" pin="VCC"/>
-<wire x1="55.88" y1="88.9" x2="55.88" y2="93.98" width="0.1524" layer="91"/>
+<pinref part="PCB1" gate="G$1" pin="VCC"/>
+<wire x1="58.42" y1="88.9" x2="55.88" y2="88.9" width="0.1524" layer="91"/>
 </segment>
 <segment>
