File: PowerSupply/PowerSupply.sch (EAGLE design)
At the start: 19 parts, among them Q2 DMMT5401, Q3 DMG2305UX

Commit message: various minor changes
Parts:
- removed C6: .47uF, SparkFun-Capacitors:CAP0805
- added C3: 47uF, SparkFun-Capacitors:CAP1210
- added JP1: M021X02_NO_SILK, SparkFun-Connectors:M021X02_NO_SILK
- C4: value (none) -> 47uF; device adafruit:CPOL-USB -> SparkFun-Capacitors:CAP1210
- C5: device SparkFun-Capacitors:CAP0805 -> SparkFun-Capacitors:CAP1210
- D1: value ssb43L -> ssa33l; device SparkFun-DiscreteSemi:DIODESMB -> SparkFun-DiscreteSemi:DIODESMA
- L1: value 4.7uH -> 15uH
Connections:
- net GND: now also C3.2, C4.2, JP1.1; no longer C4.-, C6.2
- net VCC: now also C4.1; no longer C5.1
- net VIN: now also JP1.2
- net VREG: now also C3.1, C5.1; no longer C4.+, C6.1
Other:
- note added: "GRM32ER60J476ME20L"
- note added: "VLF10040T-150M3R1"
- moved on the sheet: C1, C2, C5, D1, JP5, L1, LED1, Q2A, Q2B, Q3, R1, R2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

Commit message: Checkpointing PCB designs
Parts:
- removed SJ1: SOLDERJUMPERNO, SparkFun-Passives:SOLDERJUMPERNO
- added JP2: M02LOCK, SparkFun-Connectors:M02LOCK
- added S2: (no value), SparkFun-Electromechanical:SWITCH-SPDTPTH_LOCK
- LED1: device led:LEDCHIPLED_0805 -> adafruit:LEDCHIP-LED0805
- U$21: value DC-JACK -> DC-JACKLOWPRO; device IntegerLabs:DC-JACK -> IntegerLabs:DC-JACKLOWPRO
- U$4: VERSION v1 -> v2
Connections:
- new net N$2: JP1.2, JP5.2, S2.P, U$21.P$1
- net GND: now also JP2.1
- net VCC: now also JP2.2; no longer R2.2, SJ1.2
- net VIN: now also S2.S; no longer JP1.2, JP5.2, U$21.P$1
- net VREG: now also R2.2; no longer SJ1.1
Other:
- moved on the sheet: JP1, JP5, LED1, R2
