File: RPi/RPi.brd (EAGLE design)
At the start: 33.9 x 18 mm, 5 parts, among them X1 C-GRID-04-70553

Commit message: various minor changes
Other:
- board size 33.9 x 18 mm -> 33.5 x 18 mm
Changed lines of the file:
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@@
 <wire x1="-0.254" y1="17.78" x2="17.78" y2="17.78" width="0.254" layer="20"/>
 <wire x1="17.78" y1="17.78" x2="17.78" y2="13.97" width="0.254" layer="20"/>
-<wire x1="17.78" y1="13.97" x2="33.655" y2="13.97" width="0.254" layer="20"/>
+<wire x1="17.78" y1="13.97" x2="33.274" y2="13.97" width="0.254" layer="20"/>
 <wire x1="-0.254" y1="-0.254" x2="-0.254" y2="17.78" width="0.254" layer="20"/>
-<wire x1="-0.254" y1="-0.254" x2="33.655" y2="-0.254" width="0.254" layer="20"/>
+<wire x1="-0.254" y1="-0.254" x2="33.274" y2="-0.254" width="0.254" layer="20"/>
 <text x="17.4625" y="7.62" size="1.016" layer="21" font="vector" ratio="10" rot="R180" align="center-left">c</text>
-<wire x1="33.655" y1="13.97" x2="33.655" y2="-0.254" width="0.254" layer="20"/>
+<wire x1="33.274" y1="13.97" x2="33.274" y2="-0.254" width="0.254" layer="20"/>
 <text x="33.02" y="7.62" size="1.016" layer="21" font="vector" rot="SR0" align="center-right">Integer Labs</text>
 <text x="18.7325" y="7.62" size="1.016" layer="21" font="vector" rot="R180" align="center-right">v1</text>
@@
 <attribute name="MF" value="" x="9.8425" y="11.43" size="1.778" layer="27" font="vector" ratio="10" rot="R270" display="off"/>
 <attribute name="OC_FARNELL" value="unknown" x="9.8425" y="11.43" size="1.778" layer="27" font="vector" ratio="10" rot="R270" display="off"/>
-<attribute name="NAME" x="4.1275" y="18.0975" size="1.016" layer="25" ratio="10"/>
 </element>
 </elements>

Commit message: Checkpointing PCB designs
Parts:
- F1: value (none) -> MF-PSMF010X-2
Changed lines of the file:
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@@
 <element name="R2" library="SparkFun-Resistors" package="0805" value="" x="22.86" y="6.985" rot="MR180"/>
 <element name="U$2" library="SparkFun-Connectors" package="2X13" value="M13X22X13" x="31.75" y="3.81" smashed="yes" rot="R180"/>
-<element name="F1" library="SparkFun-Resistors" package="0805" value="" x="22.86" y="9.525" rot="MR180"/>
+<element name="F1" library="SparkFun-Resistors" package="0805" value="MF-PSMF010X-2" x="22.86" y="9.525" rot="MR180"/>
 <element name="X1" library="con-molex" package="70553-04" value="C-GRID-04-70553" x="9.8425" y="11.43" smashed="yes" rot="R270">
 <attribute name="OC_NEWARK" value="unknown" x="9.8425" y="11.43" size="1.778" layer="27" font="vector" ratio="10" rot="R270" display="off"/>
