File: RPi/RPi.sch (EAGLE design)
At the start: 5 parts, among them X1 C-GRID-04-70553

Commit message: Checkpointing PCB designs
Parts:
- F1: value (none) -> MF-PSMF010X-2
Changed lines of the file:
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@@
 <part name="R2" library="SparkFun-Resistors" deviceset="RESISTOR" device="0805-RES"/>
 <part name="U$2" library="SparkFun-Connectors" deviceset="M13X2" device="2X13"/>
-<part name="F1" library="SparkFun-Resistors" deviceset="RESISTOR" device="0805-RES"/>
+<part name="F1" library="SparkFun-Resistors" deviceset="RESISTOR" device="0805-RES" value="MF-PSMF010X-2"/>
 <part name="X1" library="con-molex" deviceset="C-GRID-04" device="-70553"/>
 </parts>
