File: SX1231/SX1231.sch (EAGLE design)
At the start: 11 parts

Commit message: Checkpointing PCB designs
Parts:
- removed B1, B3, B4, B5, B7: TACT-SWITCH, IntegerLabs:TACT-SWITCH
- removed R2: 1, SparkFun-Resistors:RESISTOR0805-RES
- added C10, C2, C5, C9: 15pF, IntegerLabs:CAP0805
- added C20, C21, C22, C8: .1uF, IntegerLabs:CAP0805
- added C3: 22pF, IntegerLabs:CAP0805
- added C4: 2.7pF, IntegerLabs:CAP0805
- added C6: .47uF, IntegerLabs:CAP0805
- added C7: 8.2pF, IntegerLabs:CAP0805
- added JP1, JP2: M01PTH, SparkFun-Connectors:M01PTH
- added L1, L4: 10nH, IntegerLabs:INDUCTOR0805
- added L2: 33nH, IntegerLabs:INDUCTOR0805
- added L3: 12nH, IntegerLabs:INDUCTOR0805
- added Q1: 32Mhz, adafruit:XTAL-4-3225
- added U$10, U$11, U$12, U$13, U$14, U$15, U$16, U$17, U$5, U$6, U$7, U$8, U$9: TESTPOINT, IntegerLabs:TESTPOINT
- added U$3: TINY841, IntegerLabs:TINY841
- added U$4: ANTENNA, IntegerLabs:ANTENNA
- added U1: (no value), SparkFun-PowerIC:MIC52053.3V
- C1: value .47uF -> 10nF; device SparkFun-Capacitors:CAP0805 -> IntegerLabs:CAP0805
- R1: device SparkFun-Passives:RESISTOR0805-RES -> IntegerLabs:RESISTOR0805
- U$1: value TINY841 -> SX1231; device IntegerLabs:TINY841 -> IntegerLabs:SX1231
- U$2: BOARD DPad -> Radio; VERSION v4 -> v1
Connections:
- removed net BUTTON0: B5.POS1, U$1.PA0
- removed net BUTTON1: B1.POS1, U$1.PA1
- removed net BUTTON2: B3.POS1, U$1.PA2
- removed net BUTTON3: B7.POS2, U$1.PA3
- removed net BUTTON4: B4.POS1, U$1.PB0
- removed net LED: R1.2, U$1.PA7
- removed net MISO: U$1.PA5, U$2.MISO
- new net +5V: U$2.VCC, U1.EN, U1.IN
- new net MISO/LED: LED1.A, U$2.MISO, U$3.PA5
- new net N$10: C3.2, C4.1, L3.2
- new net N$11: C4.2, C5.2, L3.1, L4.2
- new net N$12: C7.2, JP1.1, L4.1, U$4.ANT
- new net N$3: C9.1, Q1.X1, U$1.XTB
- new net N$4: C10.1, Q1.X2, U$1.XTA
- new net N$5: LED1.C, R1.2
- new net N$7: C22.1, U$1.VR_ANA
- new net N$9: C2.1, C3.1, L1.2, L2.2
- new net SX_DIO0: U$1.DIO0, U$5.1
- new net SX_DIO1: U$1.DIO1, U$3.PB2, U$6.1
- new net SX_DIO2: U$1.DIO2, U$3.PA7, U$7.1
- new net SX_DIO3: U$1.DIO3, U$8.1
- new net SX_DIO4: U$1.DIO4, U$9.1
- new net SX_DIO5: U$1.DIO5, U$10.1
- new net SX_MISO: U$1.MISO, U$13.1, U$3.PA0
- new net SX_MOSI: U$1.MOSI, U$14.1, U$3.PA1
- new net SX_NSS: U$1.NSS, U$15.1, U$3.PA2
- new net SX_RESET: U$1.RESET, U$11.1, U$3.PB0
- new net SX_RXTX: U$1.RXTX, U$17.1, U$3.PB1
- new net SX_SCK: U$1.SCK, U$16.1, U$3.PA3
- new net VR_PA: C1.1, L2.1, U$1.VR_PA
- net GND: now also C1.2, C10.2, C2.2, C20.2, C21.2, C22.2, C5.1, C6.1, C7.1, C8.2, C9.2, R1.1, U$12.1, U$3.GND, U1.GND; no longer B1.NEG2, B3.NEG2, B4.NEG2, B5.NEG2, B7.NEG2, C1.1, LED1.C
- net N$2: now also C8.1, U$1.VR_DIG; no longer R2.2, U$2.VCC
- net N$8: now also L1.1, U$1.RFIO; no longer LED1.A, R1.1
- net RESET: now also U$3.PB3; no longer U$1.PB3
- net SCL/SCK: now also U$3.PA4; no longer U$1.PA4
- net SDA/MOSI: now also U$3.PA6; no longer U$1.PA6
- net VCC: now also C20.1, C21.1, C6.2, U$1.VBAT1, U$1.VBAT2, U$3.VCC, U1.OUT; no longer C1.2, R2.1, U$1.VCC
Other:
- moved on the sheet: C1, LED1, R1
