File: ColorDisplay/ColorDisplay.sch (EAGLE design)
At the start: 16 parts, among them SW1 7914J-1-000E, SW2 7914J-1-000E, SW3 7914J-1-000E, U1 ER-OLED0.95-2C, U2 LM2665M6/NOPB, U3 ATSAMD21E18A-AU, U4 MIC5205-3.3YM5 TR

Commit message: Various updates
Parts:
- removed C5: 10uF, Modulo:CAPACITOR
- removed C6: .47uF, Modulo:CAPACITOR
- C1, C2: device Modulo:CAPACITOR -> Modulo:CAPACITOR-10UF-1206
- C4: value 10uF -> 100nF; device Modulo:CAPACITOR -> Modulo:CAPACITOR-100NF
- D1: PARTNUM (none) -> SSA33L-E3/61T
- PCB1: value EXCLUDE -> DEVICE-PCB-TABS; device Modulo:DEVICE-PCB -> Modulo:DEVICE-PCB-TABS
- R1: device Modulo:RESISTOR -> Modulo:RESISTOR-0603
- U1: value ER-OLED0.95-2C -> LM2665M6/NOPB; device Modulo:OLED-COLORREVERSE -> Modulo:LM2665; SUPPLIER buydisplay.com -> (none)
- U2: value LM2665M6/NOPB -> ER-OLED0.95-2C; device Modulo:LM2665 -> Modulo:OLED-COLORREVERSE; SUPPLIER (none) -> buydisplay.com
Connections:
- net +10V: now also U1.OUT, U2.VCC; no longer U1.VCC, U2.OUT
- net +3.3V: now also C4.1, U2.VDD, U2.VDDIO; no longer C5.1, C6.1, U1.VDD, U1.VDDIO
- net +5V: now also U1.V+; no longer C4.1, U2.V+
- net BS0: now also U2.BS2; no longer U1.BS2
- net BS1: now also U2.BS1; no longer U1.BS1
- net BUTTON1: now also SW1.POS1; no longer SW2.POS1
- net BUTTON2: now also SW2.POS1; no longer SW3.POS1
- net BUTTON3: now also SW3.POS1; no longer SW1.POS1
- net CS: now also U2.CS; no longer U1.CS
- net D/C: now also U2.D/C; no longer U1.D/C
- net D0: now also U2.D0; no longer U1.D0
- net D1: now also U2.D1; no longer U1.D1
- net D2: now also U2.D2; no longer U1.D2
- net D3: now also U2.D3; no longer U1.D3
- net D4: now also U2.D4; no longer U1.D4
- net D5: now also U2.D5; no longer U1.D5
- net D6: now also U2.D6; no longer U1.D6
- net D7: now also U2.D7; no longer U1.D7
- net DISPLAY_RESET: now also U2.RESET; no longer U1.RESET
- net GND: now also U1.GND, U1.SD, U2.VSS; no longer C5.2, C6.2, U1.VSS, U2.GND, U2.SD
- net N$13: now also U1.CAP+; no longer U2.CAP+
- net N$14: now also U1.CAP-; no longer U2.CAP-
- net N$5: now also U2.VCOMH; no longer U1.VCOMH
- net N$8: now also U2.IREF; no longer U1.IREF
- net RD: now also U2.E; no longer U1.E
- net WR: now also U2.R/W; no longer U1.R/W
Other:
- moved on the sheet: C1, C2, C4, SW1, SW2, SW3
