File: PerfBoard/PerfBoard.brd (EAGLE design)
At the start: 36.3 x 29.8 mm, 32 parts

Commit message: Various updates
Parts:
- removed F1: (no value), IntegerLabs:0805
- removed U$2: TINY841, IntegerLabs:SOIC14
- removed U$4, U$6: (no value), SparkFun-Connectors:1X03_NO_SILK
- added JP13: (no value), SparkFun-Connectors:1X05_NO_SILK
- added JP18: (no value), SparkFun-Connectors:1X03_NO_SILK
- added U1: ATTINY841, Modulo:SOIC-14
- C1: value (none) -> 100nF; device IntegerLabs:0805 -> Modulo:0603
- JP10, JP11, JP7: device SparkFun-Connectors:1X05_NO_SILK -> SparkFun-Connectors:1X03_NO_SILK
- JP2, JP5: device SparkFun-Connectors:1X03_NO_SILK -> SparkFun-Connectors:1X05_NO_SILK
- LED1: value (none) -> blue; device adafruit:CHIP-LED0805 -> Modulo:0805-LED
- PCB1: value FOOTPRINTFOOTPRINT-2 -> EXCLUDE
- R1, R2, R4, R5, R6, R7, R8, R9: value 130 -> 150Ω; device IntegerLabs:0805 -> Modulo:0603
- R3: value (none) -> 681Ω; device IntegerLabs:0805 -> Modulo:0603
- moved R8 24.9 mm to (20.3, 25.1), turned to 270 degrees
- moved R9 24.9 mm to (5.08, 5.40), turned to 90 degrees
- moved JP10 18.0 mm to (20.3, 20.3), turned to 270 degrees
- moved JP11 18.0 mm to (27.9, 20.3), turned to 270 degrees
- moved JP5 18.0 mm to (17.8, 2.54), turned to 90 degrees
- moved JP7 18.0 mm to (17.8, 20.3), turned to 270 degrees
- moved JP4 17.0 mm to (15.2, 20.3)
- moved JP6 14.8 mm to (10.2, 7.62)
- moved JP2 5.68 mm to (15.2, 2.54), turned to 90 degrees
- moved JP12 2.54 mm to (25.4, 2.54)
- moved JP3 2.54 mm to (12.7, 7.62)
- moved JP8 2.54 mm to (20.3, 2.54)
- moved JP9 2.54 mm to (22.9, 2.54)
- renumbered U$1 to JP17, U$3 to PCB1, U$5 to JP14, U$7 to JP15, U$8 to JP16
Connections:
- removed net N$1: F1.2, PCB1.BUS2
- net A0: now also U1.13; no longer U$2.13
- net A1: now also U1.12; no longer U$2.12
- net A2: now also R8.1, U1.11; no longer R9.1, U$2.11
- net A3: now also U1.10; no longer U$2.10
- net A7: now also U1.6; no longer U$2.6
- net B0: now also R9.1, U1.2; no longer R8.1, U$2.2
- net B1: now also U1.3; no longer U$2.3
- net B2: now also U1.5; no longer U$2.5
- net GND: now also JP7.1, U1.14; no longer JP6.1, U$2.14
- net LED/MISO: now also U1.8; no longer U$2.8
- net N$11: now also R8.2; no longer R9.2
- net N$12: now also R9.2; no longer R8.2
- net N$3: now also JP3.1; no longer JP2.1
- net N$4: now also JP6.1; no longer JP3.1
- net N$6: now also JP10.1; no longer U$4.1
- net N$7: now also JP11.1; no longer U$6.1
- net RESET: now also U1.4; no longer U$2.4
- net SCL/SCK: now also U1.9; no longer U$2.9
- net SDA/MOSI: now also U1.7; no longer U$2.7
- net VCC: now also JP4.1, PCB1.BUS2, U1.1; no longer F1.1, JP5.1, U$2.1
Routing:
- net N$1: track 8.33 -> 0.00 mm, vias 1 -> 0
