File: PerfBoard/PerfBoard.sch (EAGLE design)
At the start: 32 parts

Commit message: Various updates
Parts:
- removed F1: (no value), IntegerLabs:RESISTOR0805
- removed U$2: TINY841, IntegerLabs:TINY841
- removed U$4, U$6: (no value), SparkFun-Connectors:M031X03_NO_SILK
- added JP13: (no value), SparkFun-Connectors:M05NO_SILK
- added JP18: (no value), SparkFun-Connectors:M031X03_NO_SILK
- added U1: ATTINY841, Modulo:ATTINY841
- C1: value (none) -> 100nF; device IntegerLabs:CAP0805 -> Modulo:CAPACITOR-100NF
- JP10, JP11, JP7: device SparkFun-Connectors:M05NO_SILK -> SparkFun-Connectors:M031X03_NO_SILK
- JP2, JP5: device SparkFun-Connectors:M031X03_NO_SILK -> SparkFun-Connectors:M05NO_SILK
- LED1: value (none) -> blue; device adafruit:LEDCHIP-LED0805 -> Modulo:LED-0805-BLUE
- PCB1: value FOOTPRINTFOOTPRINT-2 -> EXCLUDE
- R1, R2, R4, R5, R6, R7, R8, R9: value 130 -> 150Ω; device IntegerLabs:RESISTOR0805 -> Modulo:RESISTOR-150Ω
- R3: value (none) -> 681Ω; device IntegerLabs:RESISTOR0805 -> Modulo:RESISTOR-681Ω
- renumbered U$1 to JP17, U$3 to PCB1, U$5 to JP14, U$7 to JP15, U$8 to JP16
Connections:
- removed net N$1: F1.2, PCB1.VCC
- net A0: now also U1.PA0; no longer U$2.PA0
- net A1: now also U1.PA1; no longer U$2.PA1
- net A2: now also R8.1, U1.PA2; no longer R9.1, U$2.PA2
- net A3: now also U1.PA3; no longer U$2.PA3
- net A7: now also U1.PA7; no longer U$2.PA7
- net B0: now also R9.1, U1.PB0; no longer R8.1, U$2.PB0
- net B1: now also U1.PB1; no longer U$2.PB1
- net B2: now also U1.PB2; no longer U$2.PB2
- net GND: now also JP7.1, U1.GND; no longer JP6.1, U$2.GND
- net LED/MISO: now also U1.PA5; no longer U$2.PA5
- net N$11: now also R8.2; no longer R9.2
- net N$12: now also R9.2; no longer R8.2
- net N$3: now also JP3.1; no longer JP2.1
- net N$4: now also JP6.1; no longer JP3.1
- net N$6: now also JP10.1; no longer U$4.1
- net N$7: now also JP11.1; no longer U$6.1
- net RESET: now also U1.PB3; no longer U$2.PB3
- net SCL/SCK: now also U1.PA4; no longer U$2.PA4
- net SDA/MOSI: now also U1.PA6; no longer U$2.PA6
- net VCC: now also JP4.1, PCB1.VCC, U1.VCC; no longer F1.1, JP5.1, U$2.VCC
Other:
- moved on the sheet: JP12, JP3, JP4, JP6, JP8, JP9, R8, R9
