File: Old/MagKnob/Knob.sch (EAGLE design)
At the start: 10 parts, among them SW1 TopUp EC12PLRGBSDVBF-D, U1 attiny841-ssur

Commit message: Moved a bunch of files around
Parts:
- LED1: value LTST-C171TBKT -> blue
- PCB1: value MAGDEVICE -> MAGDEVICE-V2; device Modulo:MAGDEVICE -> Modulo:MAGDEVICE-V2
- SW1: device SparkFun-Electromechanical:ENCODER_RGB_CA -> Modulo:ENCODER_RGB_CA
Changed lines of the file:
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@@
 <parts>
 <part name="R2" library="Modulo" deviceset="RESISTOR" device="" value="680"/>
-<part name="LED1" library="Modulo" deviceset="LED" device="-0805-BLUE" value="LTST-C171TBKT"/>
-<part name="SW1" library="SparkFun-Electromechanical" deviceset="ENCODER_RGB_CA" device="" value="TopUp EC12PLRGBSDVBF-D"/>
+<part name="LED1" library="Modulo" deviceset="LED" device="-0805-BLUE" value="blue"/>
+<part name="SW1" library="Modulo" deviceset="ENCODER_RGB_CA" device="" value="TopUp EC12PLRGBSDVBF-D"/>
 <part name="R1" library="Modulo" deviceset="RESISTOR" device="" value="130"/>
 <part name="R3" library="Modulo" deviceset="RESISTOR" device="" value="68"/>
@@
 <part name="P+1" library="supply1" deviceset="VCC" device=""/>
 <part name="C2" library="Modulo" deviceset="CAPACITOR" device="" value=".47uF"/>
-<part name="PCB1" library="Modulo" deviceset="MAGDEVICE" device=""/>
+<part name="PCB1" library="Modulo" deviceset="MAGDEVICE" device="-V2" value="MAGDEVICE-V2"/>
 </parts>
 <sheets>
