File: Old/Controller/Controller.sch (EAGLE design)
At the start: 70 parts, among them Q1 16Mhz, SW1 SWITCHMJTP1234, U1 MIC5205-3.3YM5 TR, U2 ATMEGA32U4TQFP, U3 USBFCI-MICROB

Commit message: Major revision of all boards. Cleaned up old files. Exported BOM csv files for all boards
Parts:
- removed D1: DIODE-SCHOTTKY_, SparkFun-DiscreteSemi:DIODE-SCHOTTKY_
- removed JP10, JP11, JP12, JP13, JP14, JP15, JP16, JP17, JP24, JP25, JP34, JP35, JP5, JP6, JP7, JP8, JP9: M10NO_SILK, SparkFun-Connectors:M10NO_SILK
- removed JP18, JP19: (no value), SparkFun-Connectors:M05NO_SILK
- removed JP20, JP21, JP22, JP23: M01SMDNS, SparkFun-Connectors:M01SMDNS
- removed JP26, JP27, JP28: (no value), SparkFun-Connectors:M031X03_NO_SILK
- removed JP33: (no value), SparkFun-Connectors:M041X04_NO_SILK
- removed JP4: ICSP, Modulo:ICSP
- removed L1: (no value), IntegerLabs:INDUCTOR0805
- removed SJ2: (no value), SparkFun-Passives:SOLDERJUMPER_2WAYPASTE1&2
- removed U$1, U$10, U$11, U$2, U$3, U$4, U$5, U$6, U$8, U$9: HOLE#2, Modulo:HOLE#2
- removed U$7: JST-PA-TOP-SMD, Modulo:JST-PA-TOP-SMD
- added FOOTPRINT: DEVICE-PCB-TABS, Modulo:DEVICE-PCB-TABS
- added Q2: DMMT5401, IntegerLabs:TRANSISTOR-DUAL-PNP
- added Q3: DMG2305UX, transistor-power:IRLML5203
- added R12: 1.5KΩ, Modulo:RESISTOR-1.5KΩ
- added R13, R14, R15, R16, R17, R18: 150Ω, Modulo:RESISTOR-150Ω
- added R9: 47KΩ, Modulo:RESISTOR-47KΩ
- added SJ1: SOLDERJUMPERNO, SparkFun-Passives:SOLDERJUMPERNO
- C4, C7: value .1uF -> 100nF; device Modulo:CAPACITOR-.1UF -> Modulo:CAPACITOR-100NF
- C6: value .1uF -> 10uF; device Modulo:CAPACITOR-.1UF -> Modulo:CAPACITOR-10UF
- JP1: device SparkFun-Connectors:M04LOCK -> adafruit:PINHD-1X6LOCK; PARTNUM (none) -> PREC006SAAN-RC
- JP2: value M10NO_SILK -> (none); device SparkFun-Connectors:M10NO_SILK -> adafruit:PINHD-1X6LOCK; PARTNUM (none) -> PREC006SAAN-RC
- JP3: value ICSP -> (none); device Modulo:ICSP -> adafruit:PINHD-1X6LOCK; PARTNUM (none) -> PREC006SAAN-RC
- R10, R11, R8: value 4.7k -> 1.5KΩ
- R5: value 4.7k -> 10KΩ; device Modulo:RESISTOR-1.5KΩ -> Modulo:RESISTOR-10KΩ
- SW1: value SWITCHMJTP1234 -> blue; device Modulo:SWITCHMJTP1234 -> Modulo:SWITCHBOURNS-7914J
Connections:
- net VIN renamed N$3
- removed net +5V: D1.C, JP1.3, JP34.8, R7.1, SJ2.3, U$7.3, U1.EN, U1.IN
- removed net DUT_MISO: JP35.2, JP4.MISO/SWO/TDO, R8.1
- removed net DUT_MOSI: JP35.9, JP4.MOSI/TDI, R11.1
- removed net DUT_RESET: JP35.8, JP4.RESET, R5.1
- removed net DUT_RESET_5V: R5.2, U2.PB0(SS)
- removed net DUT_SCK: JP35.1, JP4.SCK/SWCLK/TCK, R10.1
- removed net DUT_SWDIO: JP35.3, JP4.SWDIO/TMS
- removed net DUT_VPROG: JP34.7, JP4.VTG
- removed net PB4: JP2.4, U2.PB4(ADC11)
- removed net PB5: JP2.5, U2.PB5(ADC12)
- removed net PB6: JP2.6, U2.PB6(ADC13)
- removed net PC6: JP2.7, U2.PC6
- removed net PC7: JP2.8, U2.PC7
- removed net PD4: JP2.1, U2.PD4(ADC8)
- removed net PD6: JP2.2, U2.PD6(ADC9)
- removed net PD7: JP2.3, U2.PD7(ADC10)
- removed net PE2: JP2.9, U2.PE2/!HWB
- new net D0: R12.2, R18.1, U2.PC7
- new net D1: R17.1, R8.2, U2.PC6
- new net D2: R10.2, R16.1, U2.PB6(ADC13)
- new net D3: R15.1, U2.PB5(ADC12)
- new net D4: R14.1, U2.PD7(ADC10)
- new net D5: R11.2, R13.1, U2.PB7
- new net N$13: JP1.2, R14.2
- new net N$14: Q2A.B, Q2A.C, Q2B.B, R5.2
- new net N$16: Q2B.C, Q3.G, R9.2
- new net N$17: JP1.3, R15.2
- new net N$18: JP1.4, R16.2
- new net N$19: JP1.5, R17.2
- new net N$20: JP1.6, R18.2
- net +3.3V: now also SJ1.2; no longer SJ2.1
- net GND: now also FOOTPRINT.GND, JP2.1, JP2.2, JP2.3, JP2.4, JP2.5, JP2.6, R5.1, R9.1; no longer JP1.1, JP3.GND, JP33.1, JP34.9, JP4.GND, U$7.1
- net LED: now also U2.PB4(ADC11); no longer U2.PE6
- net MISO: now also FOOTPRINT.MISO; no longer JP3.MISO/SWO/TDO, R11.2
- net MOSI: now also FOOTPRINT.MOSI; no longer JP3.MOSI/TDI, R8.2
- net N$10: now also R10.1
- net N$11: now also R8.1
- net N$2: now also JP1.1, R13.2; no longer C6.1, L1.2, U2.AVCC@24, U2.AVCC@44
- net N$6: now also R12.1
- net N$7: now also R11.1
- net RESET: now also FOOTPRINT.RESET; no longer JP3.RESET
- net SCK: now also FOOTPRINT.SCK; no longer JP3.SCK/SWCLK/TCK, R10.2
- net SCL: now also FOOTPRINT.SCL; no longer JP1.4, JP34.2, U$7.4
- net SDA: now also FOOTPRINT.SDA; no longer JP1.2, JP34.1, U$7.2
- net VBUS: now also C6.1, Q2A.E, Q3.D; no longer D1.A
- net VCC: now also FOOTPRINT.VCC, FOOTPRINT.VPROG, JP3.1, JP3.2, JP3.3, JP3.4, JP3.5, JP3.6, Q2B.E, Q3.S, R7.1, SJ1.1, U1.EN, U1.IN, U2.AVCC@24, U2.AVCC@44; no longer JP2.10, JP3.VTG, L1.1, SJ2.2
Other:
- note removed: "Perf Board Area"
- note removed: "Pogo Pin Holes"
- note removed: "programming connector 32u4"
- note removed: "programming connector for dut note that miso and mosi are switched"
- moved on the sheet: C1, C2, C3, C4, C5, C6, C7, F1, LED1, LED2, R1, R10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
