File: ParticleBase/ParticleBase.sch (EAGLE design)
At the start: 29 parts

Commit message: Fixed 3.3V connection. The old pin worked with the Spark but not the Photon.
Connections:
- removed net N$19: JP9.1, JP9.2
- new net N$14: JP9.5, JP9.6
- net 3.3V: now also JP9.1, JP9.2; no longer JP9.5, JP9.6
Changed lines of the file:
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@@
 </segment>
 <segment>
-<pinref part="JP9" gate="G$1" pin="6"/>
-<wire x1="210.82" y1="162.56" x2="213.36" y2="162.56" width="0.1524" layer="91"/>
-<label x="213.36" y="162.56" size="1.27" layer="95" xref="yes"/>
-<pinref part="JP9" gate="G$1" pin="5"/>
-<wire x1="187.96" y1="162.56" x2="210.82" y2="162.56" width="0.1524" layer="91"/>
-<junction x="210.82" y="162.56"/>
+<pinref part="JP9" gate="G$1" pin="1"/>
+<pinref part="JP9" gate="G$1" pin="2"/>
+<wire x1="187.96" y1="167.64" x2="210.82" y2="167.64" width="0.1524" layer="91"/>
+<wire x1="210.82" y1="167.64" x2="213.36" y2="167.64" width="0.1524" layer="91"/>
+<label x="213.36" y="167.64" size="1.27" layer="95" xref="yes"/>
 </segment>
 </net>
@@
 </segment>
 </net>
-<net name="N$19" class="0">
-<segment>
-<pinref part="JP9" gate="G$1" pin="1"/>
-<pinref part="JP9" gate="G$1" pin="2"/>
-<wire x1="187.96" y1="167.64" x2="210.82" y2="167.64" width="0.1524" layer="91"/>
-</segment>
-</net>
 <net name="N$20" class="0">
 <segment>
@@
 </segment>
 </net>
+<net name="N$14" class="0">
+<segment>
+<pinref part="JP9" gate="G$1" pin="5"/>
+<pinref part="JP9" gate="G$1" pin="6"/>
+<wire x1="187.96" y1="162.56" x2="210.82" y2="162.56" width="0.1524" layer="91"/>
+</segment>
+</net>

Commit message: New Grove compatible connector footprint
Parts:
- JP2, JP4, JP7: value HEADER-1X4-JST-PA-SIDE-SMD -> HEADER-MODULO; device Modulo:HEADER-1X4-JST-PA-SIDE-SMD -> Modulo:HEADER-MODULO
Connections:
- net GND: now also JP2.GND, JP4.GND, JP7.GND; no longer JP2.1, JP4.1, JP7.1
- net SCL: now also JP2.SCL, JP4.SCL, JP7.SCL; no longer JP2.4, JP4.4, JP7.4
- net SDA: now also JP2.SDA, JP4.SDA, JP7.SDA; no longer JP2.2, JP4.2, JP7.2
- net VCC: now also JP2.VCC, JP4.VCC, JP7.VCC; no longer JP2.3, JP4.3, JP7.3
Other:
- moved on the sheet: JP2, JP4, JP7
Changed lines of the file:
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@@
 <attribute name="NOBOM" value="1"/>
 </part>
-<part name="JP4" library="Modulo" deviceset="HEADER-1X4" device="-JST-PA-SIDE-SMD" value="HEADER-1X4-JST-PA-SIDE-SMD"/>
-<part name="JP7" library="Modulo" deviceset="HEADER-1X4" device="-JST-PA-SIDE-SMD" value="HEADER-1X4-JST-PA-SIDE-SMD"/>
-<part name="JP2" library="Modulo" deviceset="HEADER-1X4" device="-JST-PA-SIDE-SMD" value="HEADER-1X4-JST-PA-SIDE-SMD"/>
 <part name="H3" library="Modulo" deviceset="HOLE" device="#2" value="HOLE#2">
 <attribute name="NOBOM" value="1"/>
@@
 <part name="H5" library="Modulo" deviceset="HOLE" device="#2"/>
 <part name="H10" library="Modulo" deviceset="HOLE" device="#2"/>
+<part name="JP7" library="Modulo" deviceset="HEADER-MODULO" device=""/>
+<part name="JP2" library="Modulo" deviceset="HEADER-MODULO" device=""/>
+<part name="JP4" library="Modulo" deviceset="HEADER-MODULO" device=""/>
 </parts>
 <sheets>
@@
 <attribute name="NOBOM" x="134.366" y="81.534" size="1.016" layer="96" display="off"/>
 </instance>
-<instance part="JP4" gate="G$1" x="71.12" y="86.36"/>
-<instance part="JP7" gate="G$1" x="101.6" y="86.36"/>
-<instance part="JP2" gate="G$1" x="33.02" y="86.36"/>
 <instance part="H3" gate="G$1" x="134.62" y="73.66">
 <attribute name="NOBOM" x="134.62" y="73.66" size="1.016" layer="96" display="off"/>
@@
 <instance part="H5" gate="G$1" x="134.62" y="58.42"/>
 <instance part="H10" gate="G$1" x="144.78" y="58.42"/>
+<instance part="JP7" gate="G$1" x="30.48" y="86.36"/>
+<instance part="JP2" gate="G$1" x="66.04" y="86.36"/>
+<instance part="JP4" gate="G$1" x="101.6" y="86.36"/>
 </instances>
 <busses>
@@
 <wire x1="101.6" y1="63.5" x2="111.76" y2="63.5" width="0.1524" layer="91"/>
 <label x="104.14" y="63.5" size="1.778" layer="95"/>
-</segment>
-<segment>
-<wire x1="96.52" y1="83.82" x2="88.9" y2="83.82" width="0.1524" layer="91"/>
-<label x="88.9" y="83.82" size="1.27" layer="95" rot="R180" xref="yes"/>
-<pinref part="JP7" gate="G$1" pin="3"/>
-</segment>
-<segment>
-<wire x1="27.94" y1="83.82" x2="20.32" y2="83.82" width="0.1524" layer="91"/>
-<label x="20.32" y="83.82" size="1.27" layer="95" rot="R180" xref="yes"/>
-<pinref part="JP2" gate="G$1" pin="3"/>
-</segment>
-<segment>
-<wire x1="66.04" y1="83.82" x2="58.42" y2="83.82" width="0.1524" layer="91"/>
-<label x="58.42" y="83.82" size="1.27" layer="95" rot="R180" xref="yes"/>
-<pinref part="JP4" gate="G$1" pin="3"/>
 </segment>
 <segment>
@@
 <junction x="139.7" y="167.64"/>
 </segment>
+<segment>
+<pinref part="JP7" gate="G$1" pin="VCC"/>
+<wire x1="22.86" y1="88.9" x2="20.32" y2="88.9" width="0.1524" layer="91"/>
+<label x="20.32" y="88.9" size="1.27" layer="95" rot="R180" xref="yes"/>
+</segment>
+<segment>
+<pinref part="JP2" gate="G$1" pin="VCC"/>
+<wire x1="58.42" y1="88.9" x2="55.88" y2="88.9" width="0.1524" layer="91"/>
+<label x="55.88" y="88.9" size="1.27" layer="95" rot="R180" xref="yes"/>
+</segment>
+<segment>
+<pinref part="JP4" gate="G$1" pin="VCC"/>
+<wire x1="93.98" y1="88.9" x2="91.44" y2="88.9" width="0.1524" layer="91"/>
+<label x="91.44" y="88.9" size="1.27" layer="95" rot="R180" xref="yes"/>
+</segment>
 </net>
 <net name="GND" class="0">
@@
 <wire x1="101.6" y1="58.42" x2="111.76" y2="58.42" width="0.1524" layer="91"/>
 <label x="104.14" y="58.42" size="1.778" layer="95"/>
-</segment>
-<segment>
-<wire x1="96.52" y1="88.9" x2="88.9" y2="88.9" width="0.1524" layer="91"/>
-<label x="88.9" y="88.9" size="1.27" layer="95" rot="R180" xref="yes"/>
-<pinref part="JP7" gate="G$1" pin="1"/>
-</segment>
-<segment>
-<wire x1="27.94" y1="88.9" x2="20.32" y2="88.9" width="0.1524" layer="91"/>
-<label x="20.32" y="88.9" size="1.27" layer="95" rot="R180" xref="yes"/>
-<pinref part="JP2" gate="G$1" pin="1"/>
-</segment>
-<segment>
-<wire x1="66.04" y1="88.9" x2="58.42" y2="88.9" width="0.1524" layer="91"/>
-<label x="58.42" y="88.9" size="1.27" layer="95" rot="R180" xref="yes"/>
-<pinref part="JP4" gate="G$1" pin="1"/>
 </segment>
 <segment>
@@
 <junction x="139.7" y="165.1"/>
 </segment>
+<segment>
+<pinref part="JP7" gate="G$1" pin="GND"/>
+<wire x1="22.86" y1="91.44" x2="20.32" y2="91.44" width="0.1524" layer="91"/>
+<label x="20.32" y="91.44" size="1.27" layer="95" rot="R180" xref="yes"/>
+</segment>
+<segment>
+<pinref part="JP2" gate="G$1" pin="GND"/>
+<wire x1="58.42" y1="91.44" x2="55.88" y2="91.44" width="0.1524" layer="91"/>
+<label x="55.88" y="91.44" size="1.27" layer="95" rot="R180" xref="yes"/>
+</segment>
+<segment>
+<pinref part="JP4" gate="G$1" pin="GND"/>
+<wire x1="93.98" y1="91.44" x2="91.44" y2="91.44" width="0.1524" layer="91"/>
+<label x="91.44" y="91.44" size="1.27" layer="95" rot="R180" xref="yes"/>
+</segment>
 </net>
 <net name="SDA" class="0">
@@
 <wire x1="33.02" y1="60.96" x2="25.4" y2="60.96" width="0.1524" layer="91"/>
 <label x="27.94" y="60.96" size="1.778" layer="95"/>
-</segment>
-<segment>
-<wire x1="96.52" y1="86.36" x2="88.9" y2="86.36" width="0.1524" layer="91"/>
-<label x="88.9" y="86.36" size="1.27" layer="95" rot="R180" xref="yes"/>
-<pinref part="JP7" gate="G$1" pin="2"/>
-</segment>
-<segment>
-<wire x1="27.94" y1="86.36" x2="20.32" y2="86.36" width="0.1524" layer="91"/>
-<label x="20.32" y="86.36" size="1.27" layer="95" rot="R180" xref="yes"/>
-<pinref part="JP2" gate="G$1" pin="2"/>
-</segment>
-<segment>
-<wire x1="66.04" y1="86.36" x2="58.42" y2="86.36" width="0.1524" layer="91"/>
-<label x="58.42" y="86.36" size="1.27" layer="95" rot="R180" xref="yes"/>
-<pinref part="JP4" gate="G$1" pin="2"/>
 </segment>
 <segment>
@@
 <junction x="210.82" y="139.7"/>
 </segment>
+<segment>
+<pinref part="JP7" gate="G$1" pin="SDA"/>
+<wire x1="22.86" y1="86.36" x2="20.32" y2="86.36" width="0.1524" layer="91"/>
+<label x="20.32" y="86.36" size="1.27" layer="95" rot="R180" xref="yes"/>
+</segment>
+<segment>
+<pinref part="JP2" gate="G$1" pin="SDA"/>
+<wire x1="58.42" y1="86.36" x2="55.88" y2="86.36" width="0.1524" layer="91"/>
+<label x="55.88" y="86.36" size="1.27" layer="95" rot="R180" xref="yes"/>
+</segment>
+<segment>
+<pinref part="JP4" gate="G$1" pin="SDA"/>
+<wire x1="93.98" y1="86.36" x2="91.44" y2="86.36" width="0.1524" layer="91"/>
+<label x="91.44" y="86.36" size="1.27" layer="95" rot="R180" xref="yes"/>
+</segment>
 </net>
 <net name="SCL" class="0">
@@
 <wire x1="25.4" y1="66.04" x2="33.02" y2="66.04" width="0.1524" layer="91"/>
 <label x="27.94" y="66.04" size="1.778" layer="95"/>
-</segment>
-<segment>
-<wire x1="96.52" y1="81.28" x2="88.9" y2="81.28" width="0.1524" layer="91"/>
-<label x="88.9" y="81.28" size="1.27" layer="95" rot="R180" xref="yes"/>
-<pinref part="JP7" gate="G$1" pin="4"/>
-</segment>
-<segment>
-<wire x1="27.94" y1="81.28" x2="20.32" y2="81.28" width="0.1524" layer="91"/>
-<label x="20.32" y="81.28" size="1.27" layer="95" rot="R180" xref="yes"/>
-<pinref part="JP2" gate="G$1" pin="4"/>
-</segment>
-<segment>
-<wire x1="66.04" y1="81.28" x2="58.42" y2="81.28" width="0.1524" layer="91"/>
-<label x="58.42" y="81.28" size="1.27" layer="95" rot="R180" xref="yes"/>
-<pinref part="JP4" gate="G$1" pin="4"/>
 </segment>
 <segment>
@@
 <junction x="210.82" y="142.24"/>
 </segment>
+<segment>
+<pinref part="JP7" gate="G$1" pin="SCL"/>
+<wire x1="22.86" y1="83.82" x2="20.32" y2="83.82" width="0.1524" layer="91"/>
+<label x="20.32" y="83.82" size="1.27" layer="95" rot="R180" xref="yes"/>
+</segment>
+<segment>
+<pinref part="JP2" gate="G$1" pin="SCL"/>
+<wire x1="58.42" y1="83.82" x2="55.88" y2="83.82" width="0.1524" layer="91"/>
+<label x="55.88" y="83.82" size="1.27" layer="95" rot="R180" xref="yes"/>
+</segment>
+<segment>
+<pinref part="JP4" gate="G$1" pin="SCL"/>
+<wire x1="93.98" y1="83.82" x2="91.44" y2="83.82" width="0.1524" layer="91"/>
+<label x="91.44" y="83.82" size="1.27" layer="95" rot="R180" xref="yes"/>
+</segment>
 </net>

Commit message: Various updates
Parts:
- added D1, D2: RB751V40, Modulo:DIODE-SCHOTTKY-BAT60A
Connections:
- net 3.3V: now also D1.C, D2.C
- net SCL: now also D1.A
- net SDA: now also D2.A
Other:
- moved on the sheet: R2
Changed lines of the file:
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@@
 <part name="JP2" library="Modulo" deviceset="HEADER-MODULO" device=""/>
 <part name="JP4" library="Modulo" deviceset="HEADER-MODULO" device=""/>
+<part name="D1" library="Modulo" deviceset="DIODE-SCHOTTKY" device="-BAT60A" value="RB751V40">
+<attribute name="PARTNUM" value="RB751V40"/>
+</part>
+<part name="D2" library="Modulo" deviceset="DIODE-SCHOTTKY" device="-BAT60A" value="RB751V40">
+<attribute name="PARTNUM" value="RB751V40"/>
+</part>
 </parts>
 <sheets>
@@
 <attribute name="BOM" x="40.64" y="127" size="1.778" layer="96" display="off"/>
 </instance>
-<instance part="R2" gate="G$1" x="78.74" y="137.16" rot="R90"/>
+<instance part="R2" gate="G$1" x="91.44" y="137.16" rot="R90"/>
 <instance part="R1" gate="G$1" x="73.66" y="137.16" rot="R90"/>
 <instance part="C1" gate="G$1" x="40.64" y="139.7"/>
@@
 <instance part="JP2" gate="G$1" x="66.04" y="86.36"/>
 <instance part="JP4" gate="G$1" x="101.6" y="86.36"/>
+<instance part="D1" gate="G$1" x="81.28" y="137.16" rot="R270"/>
+<instance part="D2" gate="G$1" x="99.06" y="137.16" rot="R270"/>
 </instances>
 <busses>
@@
 </segment>
 <segment>
-<label x="81.28" y="147.32" size="1.778" layer="95" xref="yes"/>
+<label x="101.6" y="147.32" size="1.778" layer="95" xref="yes"/>
 <pinref part="R2" gate="G$1" pin="2"/>
-<wire x1="78.74" y1="147.32" x2="81.28" y2="147.32" width="0.1524" layer="91"/>
-<wire x1="78.74" y1="142.24" x2="78.74" y2="147.32" width="0.1524" layer="91"/>
+<wire x1="91.44" y1="147.32" x2="101.6" y2="147.32" width="0.1524" layer="91"/>
+<wire x1="91.44" y1="142.24" x2="91.44" y2="144.78" width="0.1524" layer="91"/>
+<pinref part="D2" gate="G$1" pin="A"/>
+<wire x1="91.44" y1="144.78" x2="91.44" y2="147.32" width="0.1524" layer="91"/>
+<wire x1="99.06" y1="139.7" x2="99.06" y2="144.78" width="0.1524" layer="91"/>
+<wire x1="99.06" y1="144.78" x2="91.44" y2="144.78" width="0.1524" layer="91"/>
 </segment>
 <segment>
@@
 <pinref part="R1" gate="G$1" pin="2"/>
 <wire x1="73.66" y1="152.4" x2="81.28" y2="152.4" width="0.1524" layer="91"/>
-<wire x1="73.66" y1="142.24" x2="73.66" y2="152.4" width="0.1524" layer="91"/>
+<wire x1="73.66" y1="142.24" x2="73.66" y2="147.32" width="0.1524" layer="91"/>
+<pinref part="D1" gate="G$1" pin="A"/>
+<wire x1="73.66" y1="147.32" x2="73.66" y2="152.4" width="0.1524" layer="91"/>
+<wire x1="81.28" y1="139.7" x2="81.28" y2="147.32" width="0.1524" layer="91"/>
+<wire x1="81.28" y1="147.32" x2="73.66" y2="147.32" width="0.1524" layer="91"/>
 </segment>
 <segment>
@@
 <segment>
 <pinref part="R2" gate="G$1" pin="1"/>
-<wire x1="78.74" y1="132.08" x2="78.74" y2="127" width="0.1524" layer="91"/>
+<wire x1="91.44" y1="132.08" x2="91.44" y2="127" width="0.1524" layer="91"/>
 <pinref part="R1" gate="G$1" pin="1"/>
-<wire x1="78.74" y1="127" x2="73.66" y2="127" width="0.1524" layer="91"/>
+<wire x1="91.44" y1="127" x2="81.28" y2="127" width="0.1524" layer="91"/>
+<wire x1="81.28" y1="127" x2="73.66" y2="127" width="0.1524" layer="91"/>
 <wire x1="73.66" y1="127" x2="73.66" y2="132.08" width="0.1524" layer="91"/>
 <wire x1="73.66" y1="127" x2="68.58" y2="127" width="0.1524" layer="91"/>
 <label x="68.58" y="127" size="1.778" layer="95" rot="R180" xref="yes"/>
 <junction x="73.66" y="127"/>
-</segment>
-<segment>
+<pinref part="D1" gate="G$1" pin="C"/>
+<wire x1="81.28" y1="134.62" x2="81.28" y2="127" width="0.1524" layer="91"/>
+<pinref part="D2" gate="G$1" pin="C"/>
+<wire x1="91.44" y1="127" x2="99.06" y2="127" width="0.1524" layer="91"/>
+<wire x1="99.06" y1="127" x2="99.06" y2="134.62" width="0.1524" layer="91"/>
+</segment>
+<segment>

Commit message: Various small tweaks based on testing and feedback from manufacturer.
Parts:
- added C2: 10uF, Modulo:CAPACITOR-10UF
- added R3, R4: 12Ω, Modulo:RESISTOR-12Ω
- added U1: VREG-MIC5205-3.3V, Modulo:VREG-MIC5205-3.3V
- JP8, JP9: PARTNUM (none) -> 12x2 Receptacle
- R1, R2: value 1KΩ -> 5kΩ; device Modulo:RESISTOR-1KΩ -> Modulo:RESISTOR-5KΩ
Connections:
- new net N$16: D1.C, R3.2
- new net N$19: D2.C, R4.2
- new net N$34: JP9.1, JP9.2
- net 3.3V: now also C2.2, R3.1, R4.1, U1.OUT; no longer D1.C, D2.C, JP9.1, JP9.2
- net GND: now also C2.1, U1.GND
- net VCC: now also U1.EN, U1.IN
Other:
- note added: "We have our own 3.3v regulator, even though the particle board can provide 3.3v, to ensure that clamping to 3.3v and pullup resistors work when particle is not attached"
- moved on the sheet: D1, D2

Commit message: Various minor tweaks based on testing and feedback from manufacturer
Parts:
- added SJ1: SOLDERJUMPERNO, SparkFun-Passives:SOLDERJUMPERNO
Connections:
- net 3.3V: now also SJ1.2
- net N$34: now also SJ1.1
Changed lines of the file:
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@@
 <part name="U1" library="Modulo" deviceset="VREG-MIC5205" device="-3.3V"/>
 <part name="C2" library="Modulo" deviceset="CAPACITOR" device="-10UF" value="10uF"/>
+<part name="SJ1" library="SparkFun-Passives" deviceset="SOLDERJUMPER" device="NO"/>
 </parts>
 <sheets>
@@
 <instance part="U1" gate="G$1" x="71.12" y="33.02"/>
 <instance part="C2" gate="G$1" x="71.12" y="48.26" rot="R90"/>
+<instance part="SJ1" gate="1" x="220.98" y="167.64"/>
 </instances>
 <busses>
@@
 <label x="83.82" y="48.26" size="1.778" layer="95" xref="yes"/>
 </segment>
+<segment>
+<pinref part="SJ1" gate="1" pin="2"/>
+<wire x1="226.06" y1="167.64" x2="231.14" y2="167.64" width="0.1524" layer="91"/>
+<label x="231.14" y="167.64" size="1.778" layer="95" xref="yes"/>
+</segment>
 </net>
 <net name="N$1" class="0">
@@
 <pinref part="JP9" gate="G$1" pin="2"/>
 <wire x1="187.96" y1="167.64" x2="210.82" y2="167.64" width="0.1524" layer="91"/>
-</segment>
-</net>
+<pinref part="SJ1" gate="1" pin="1"/>
+<wire x1="215.9" y1="167.64" x2="210.82" y2="167.64" width="0.1524" layer="91"/>
+</segment>
+</net>

Commit message: Added unique board prefixes to part numbers due to CM requirements
Parts:
- added 1-FOOT1, 1-FOOT2, 1-FOOT3, 1-FOOT4: FOOT, Modulo:FOOT
- renumbered C1 to 1-C1, C2 to 1-C2, D1 to 1-D1, D2 to 1-D2, G1 to 1-G1, G2 to 1-G2, G3 to 1-G3, JP1 to 1-JP1, JP2 to 1-JP2, JP3 to 1-JP3, JP4 to 1-JP4, JP5 to 1-JP5, JP6 to 1-JP6, JP7 to 1-JP7, JP8 to 1-JP8, JP9 to 1-JP9, R1 to 1-R1, R2 to 1-R2, R3 to 1-R3, R4 to 1-R4, SJ1 to 1-SJ1, U1 to 1-U1
